Commit message: add finger tip to urdf for better retargeting

File: examples/retarget_helpers/hand/xarm/xarm7_standalone.urdf (robot description, URDF)
Before this commit: robot UF_ROBOT, 18 links, 17 joints
Links:
- added link left_tip
- added link right_tip
Joints:
- added joint left_tip_joint: type fixed, parent left_finger, child left_tip, origin xyz=0 -0.026 0.061 rpy=0 0 0
- added joint right_tip_joint: type fixed, parent right_finger, child right_tip, origin xyz=0 0.026 0.061 rpy=0 0 0
