Commit message: Retargeting complete, will work on arm integration

File: src/retarget_helpers/hand/ruka/robot.urdf (robot description, URDF)
Before this commit: robot folderv2, 27 links, 26 joints
Joints:
- joint thumb_mcp: limit lower=-0.77 upper=0.7 effort=10 velocity=10 -> lower=-0.77 upper=1.57 effort=10 velocity=10
